File: HardGFX_STM32H745/HardGFX_Debug.sch (KiCad schematic (older format))
At the start: 3 parts, among them J4 Conn_ARM_JTAG_SWD_10

Commit message: Filling field for do BOM with Kicost  and create proyect on IDE to start setting peripheral in MCU
Parts:
- CR3: renamed from CR2; Digikey# (none) -> 497-7231-1-ND; MANUFACTURER (none) -> STMicroelectronics; Manf# (none) -> ESDALC6V1W5; Mouser# (none) -> 511-ESDALC6V1W5
- CR4: renamed from CR3; Digikey# (none) -> 497-7231-1-ND; MANUFACTURER (none) -> STMicroelectronics; Manf# (none) -> ESDALC6V1W5; Mouser# (none) -> 511-ESDALC6V1W5
- renumbered J4 to J3
Changed lines of the file:
@@
 $EndDescr
 $Comp
-L Connector:Conn_ARM_JTAG_SWD_10 J4
+L Connector:Conn_ARM_JTAG_SWD_10 J3
 U 1 1 60C12D28
 P 4350 3000
-F 0 "J4" H 3907 3046 50  0000 R CNN
+F 0 "J3" H 3907 3046 50  0000 R CNN
 F 1 "Conn_ARM_JTAG_SWD_10" H 3907 2955 50  0000 R CNN
 F 2 "Connector_PinHeader_1.27mm:PinHeader_2x05_P1.27mm_Vertical" H 4350 3000 50  0001 C CNN
@@
 $EndComp
 $Comp
-L power:+3V3 #PWR029
+L power:+3V3 #PWR038
 U 1 1 60C13851
 P 4350 2250
-F 0 "#PWR029" H 4350 2100 50  0001 C CNN
+F 0 "#PWR038" H 4350 2100 50  0001 C CNN
 F 1 "+3V3" H 4365 2423 50  0000 C CNN
 F 2 "" H 4350 2250 50  0001 C CNN
@@
 	4350 2250 4350 2400
 $Comp
-L power:GNDD #PWR030
+L power:GNDD #PWR039
 U 1 1 60C1415D
 P 4350 3800
-F 0 "#PWR030" H 4350 3550 50  0001 C CNN
+F 0 "#PWR039" H 4350 3550 50  0001 C CNN
 F 1 "GNDD" H 4354 3645 50  0000 C CNN
 F 2 "" H 4350 3800 50  0001 C CNN
@@
 NJTRST
 $Comp
-L ESDALC6V1W5:ESDALC6V1W5 CR2
+L ESDALC6V1W5:ESDALC6V1W5 CR3
 U 1 1 60C17A05
 P 4400 5150
-F 0 "CR2" H 4150 5500 60  0000 L CNN
+F 0 "CR3" H 4150 5500 60  0000 L CNN
 F 1 "ESDALC6V1W5" H 4150 5400 60  0000 L CNN
 F 2 "ESDALC6V1W5:ESDALC6V1W5" V 4700 5450 60  0001 C CNN
 F 3 "https://www.st.com/resource/en/datasheet/esdalc6v1w.pdf" H 4400 5150 60  0001 C CNN
+F 4 "497-7231-1-ND" H 4400 5150 50  0001 C CNN "Digikey#"
+F 5 "STMicroelectronics" H 4400 5150 50  0001 C CNN "MANUFACTURER"
+F 6 "ESDALC6V1W5" H 4400 5150 50  0001 C CNN "Manf#"
+F 7 "511-ESDALC6V1W5" H 4400 5150 50  0001 C CNN "Mouser#"
 	1    4400 5150
 	1    0    0    -1
 $EndComp
 $Comp
-L ESDALC6V1W5:ESDALC6V1W5 CR3
+L ESDALC6V1W5:ESDALC6V1W5 CR4
 U 1 1 60C1A435
 P 5400 5150
-F 0 "CR3" H 6628 5503 60  0000 L CNN
+F 0 "CR4" H 6628 5503 60  0000 L CNN
 F 1 "ESDALC6V1W5" H 6628 5397 60  0000 L CNN
 F 2 "ESDALC6V1W5:ESDALC6V1W5" V 5700 5450 60  0001 C CNN
 F 3 "https://www.st.com/resource/en/datasheet/esdalc6v1w.pdf" H 5400 5150 60  0001 C CNN
+F 4 "497-7231-1-ND" H 5400 5150 50  0001 C CNN "Digikey#"
+F 5 "STMicroelectronics" H 5400 5150 50  0001 C CNN "MANUFACTURER"
+F 6 "ESDALC6V1W5" H 5400 5150 50  0001 C CNN "Manf#"
+F 7 "511-ESDALC6V1W5" H 5400 5150 50  0001 C CNN "Mouser#"
 	1    5400 5150
 	1    0    0    -1
 $EndComp
 $Comp
-L power:GNDD #PWR031
+L power:GNDD #PWR040
 U 1 1 60C1AB4F
 P 6000 5550
-F 0 "#PWR031" H 6000 5300 50  0001 C CNN
+F 0 "#PWR040" H 6000 5300 50  0001 C CNN
 F 1 "GNDD" H 6004 5395 50  0000 C CNN
 F 2 "" H 6000 5550 50  0001 C CNN

Commit message: Almost I end to fill Kicost field on schematics.
Parts:
- J3: footprint Connector_PinHeader_1.27mm:PinHeader_2x05_P1.27mm_Vertical -> (none); Digikey# (none) -> SAM8799-ND; MANUFACTURER (none) -> Samtec; Manf# (none) -> FTSH-105-01-L-DV-K; Mouser# (none) -> 200-FTSH10501LDVK
Changed lines of the file:
@@
 Sheet 3 8
 Title "Debug JTAG"
-Date "2021-08-24"
+Date "2021-08-25"
 Rev "Rev. 1"
 Comp "HardGFX"
@@
 F 0 "J3" H 3907 3046 50  0000 R CNN
 F 1 "Conn_ARM_JTAG_SWD_10" H 3907 2955 50  0000 R CNN
-F 2 "Connector_PinHeader_1.27mm:PinHeader_2x05_P1.27mm_Vertical" H 4350 3000 50  0001 C CNN
-F 3 "" V 4000 1750 50  0001 C CNN
+F 2 "" H 4350 3000 50  0001 C CNN
+F 3 "http://suddendocs.samtec.com/catalog_english/ftsh_smt.pdf" V 4000 1750 50  0001 C CNN
+F 4 "SAM8799-ND" H 4350 3000 50  0001 C CNN "Digikey#"
+F 5 "Samtec" H 4350 3000 50  0001 C CNN "MANUFACTURER"
+F 6 "FTSH-105-01-L-DV-K" H 4350 3000 50  0001 C CNN "Manf#"
+F 7 "200-FTSH10501LDVK" H 4350 3000 50  0001 C CNN "Mouser#"
 	1    4350 3000
 	1    0    0    -1

Commit message: Modified symbols field to use Kicost
Parts:
- CR3, CR4: Manf# ESDALC6V1W5 -> (none); manf# (none) -> ESDALC6V1W5
- J3: Manf# FTSH-105-01-L-DV-K -> (none); manf# (none) -> FTSH-105-01-L-DV-K
Changed lines of the file:
@@
 F 4 "SAM8799-ND" H 4350 3000 50  0001 C CNN "Digikey#"
 F 5 "Samtec" H 4350 3000 50  0001 C CNN "MANUFACTURER"
-F 6 "FTSH-105-01-L-DV-K" H 4350 3000 50  0001 C CNN "Manf#"
-F 7 "200-FTSH10501LDVK" H 4350 3000 50  0001 C CNN "Mouser#"
+F 6 "200-FTSH10501LDVK" H 4350 3000 50  0001 C CNN "Mouser#"
+F 7 "FTSH-105-01-L-DV-K" H 4350 3000 50  0001 C CNN "manf#"
 	1    4350 3000
 	1    0    0    -1
@@
 F 4 "497-7231-1-ND" H 4400 5150 50  0001 C CNN "Digikey#"
 F 5 "STMicroelectronics" H 4400 5150 50  0001 C CNN "MANUFACTURER"
-F 6 "ESDALC6V1W5" H 4400 5150 50  0001 C CNN "Manf#"
-F 7 "511-ESDALC6V1W5" H 4400 5150 50  0001 C CNN "Mouser#"
+F 6 "511-ESDALC6V1W5" H 4400 5150 50  0001 C CNN "Mouser#"
+F 7 "ESDALC6V1W5" H 4400 5150 50  0001 C CNN "manf#"
 	1    4400 5150
 	1    0    0    -1
@@
 F 4 "497-7231-1-ND" H 5400 5150 50  0001 C CNN "Digikey#"
 F 5 "STMicroelectronics" H 5400 5150 50  0001 C CNN "MANUFACTURER"
-F 6 "ESDALC6V1W5" H 5400 5150 50  0001 C CNN "Manf#"
-F 7 "511-ESDALC6V1W5" H 5400 5150 50  0001 C CNN "Mouser#"
+F 6 "511-ESDALC6V1W5" H 5400 5150 50  0001 C CNN "Mouser#"
+F 7 "ESDALC6V1W5" H 5400 5150 50  0001 C CNN "manf#"
 	1    5400 5150
 	1    0    0    -1
