File: HardGFX_STM32H745/HardGFX_LCD.sch (KiCad schematic (older format))
At the start: 18 parts, among them J5 ER-CON40HT-1, J6 ER-CON10HT-1, U5 TPS61165DRVR

Commit message: Filling field for do BOM with Kicost  and create proyect on IDE to start setting peripheral in MCU
Parts:
- D2: Digikey# (none) -> ZHCS400CT-ND; MANUFACTURER (none) -> Diodes Incorporated; Manf# (none) -> ZHCS400TA; Mouser# (none) -> 522-ZHCS400TA
- U5: Digikey# (none) -> 2156-TPS61165DRVR-ND; MANUFACTURER (none) -> Texas Instruments; Manf# (none) -> TPS61165DRVR; Mouser# (none) -> 595-TPS61165DRVR
- renumbered C38 to C42, C39 to C43, C40 to C44, C41 to C45, C42 to C46, C43 to C47, C44 to C48, J5 to J4, J6 to J5, R3 to R8, R4 to R9
Changed lines of the file:
@@
 $EndDescr
 $Comp
-L power:+3V3 #PWR036
+L power:+3V3 #PWR046
 U 1 1 60DF7FCC
 P 3700 3300
-F 0 "#PWR036" H 3700 3150 50  0001 C CNN
+F 0 "#PWR046" H 3700 3150 50  0001 C CNN
 F 1 "+3V3" H 3715 3473 50  0000 C CNN
 F 2 "" H 3700 3300 50  0001 C CNN
@@
 	3700 3750 3700 3700
 $Comp
-L power:GNDD #PWR037
+L power:GNDD #PWR047
 U 1 1 60DF57CC
 P 3700 3750
-F 0 "#PWR037" H 3700 3500 50  0001 C CNN
+F 0 "#PWR047" H 3700 3500 50  0001 C CNN
 F 1 "GNDD" H 3704 3595 50  0000 C CNN
 F 2 "" H 3700 3750 50  0001 C CNN
@@
 	3550 3400 3700 3400
 $Comp
-L Device:C C40
+L Device:C C44
 U 1 1 60DE6828
 P 3550 3550
-F 0 "C40" H 3200 3600 50  0000 L CNN
+F 0 "C44" H 3200 3600 50  0000 L CNN
 F 1 "100nF" H 3200 3500 50  0000 L CNN
 F 2 "Capacitor_SMD:C_0603_1608Metric" H 3588 3400 50  0001 C CNN
@@
 LCD_DISP
 $Comp
-L Device:R R4
+L Device:R R9
 U 1 1 60D78415
 P 5000 6600
-F 0 "R4" H 5070 6646 50  0000 L CNN
+F 0 "R9" H 5070 6646 50  0000 L CNN
 F 1 "4.7K" H 5070 6555 50  0000 L CNN
 F 2 "" V 4930 6600 50  0001 C CNN
@@
 	5500 6550 5300 6550
 $Comp
-L power:GNDD #PWR038
+L power:GNDD #PWR048
 U 1 1 60D73142
 P 5150 6850
-F 0 "#PWR038" H 5150 6600 50  0001 C CNN
+F 0 "#PWR048" H 5150 6600 50  0001 C CNN
 F 1 "GNDD" H 5154 6695 50  0000 C CNN
 F 2 "" H 5150 6850 50  0001 C CNN
@@
 NoConn ~ 5500 6950
 $Comp
-L ER-CON40HT-1:ER-CON40HT-1 J5
+L ER-CON40HT-1:ER-CON40HT-1 J4
 U 1 1 60D5B202
 P 5500 3100
-F 0 "J5" H 6330 1246 50  0000 L CNN
+F 0 "J4" H 6330 1246 50  0000 L CNN
 F 1 "ER-CON40HT-1" H 6330 1155 50  0000 L CNN
 F 2 "ER-CONNECTOR:ER-CON40HT-1" H 5500 3100 50  0001 L BNN
@@
 	9500 3200 9650 3200
 $Comp
-L power:GNDD #PWR042
+L power:GNDD #PWR052
 U 1 1 60D66B06
 P 9650 3300
-F 0 "#PWR042" H 9650 3050 50  0001 C CNN
+F 0 "#PWR052" H 9650 3050 50  0001 C CNN
 F 1 "GNDD" H 9654 3145 50  0000 C CNN
 F 2 "" H 9650 3300 50  0001 C CNN
@@
 $EndComp
 $Comp
-L Device:C C43
+L Device:C C47
 U 1 1 60D64498
 P 9500 3050
-F 0 "C43" H 9200 3100 50  0000 L CNN
+F 0 "C47" H 9200 3100 50  0000 L CNN
 F 1 "100nF" H 9150 3000 50  0000 L CNN
 F 2 "Capacitor_SMD:C_0603_1608Metric" H 9538 2900 50  0001 C CNN
@@
 	8800 4400 8950 4400
 $Comp
-L power:GNDD #PWR040
+L power:GNDD #PWR050
 U 1 1 60D5E77C
 P 8950 4500
-F 0 "#PWR040" H 8950 4250 50  0001 C CNN
+F 0 "#PWR050" H 8950 4250 50  0001 C CNN
 F 1 "GNDD" H 8954 4345 50  0000 C CNN
 F 2 "" H 8950 4500 50  0001 C CNN
@@
 $EndComp
 $Comp
-L power:+3V3 #PWR041
+L power:+3V3 #PWR051
 U 1 1 60D5E1CB
 P 9650 2800
-F 0 "#PWR041" H 9650 2650 50  0001 C CNN
+F 0 "#PWR051" H 9650 2650 50  0001 C CNN
 F 1 "+3V3" H 9665 2973 50  0000 C CNN
 F 2 "" H 9650 2800 50  0001 C CNN
@@
 	7700 3700 7700 3600
 $Comp
-L power:GNDD #PWR039
+L power:GNDD #PWR049
 U 1 1 60D5D40A
 P 7700 3700
-F 0 "#PWR039" H 7700 3450 50  0001 C CNN
+F 0 "#PWR049" H 7700 3450 50  0001 C CNN
 F 1 "GNDD" H 7704 3545 50  0000 C CNN
 F 2 "" H 7700 3700 50  0001 C CNN
@@
 $EndComp
 $Comp
-L ER-CON10HT-1:ER-CON10HT-1 J6
+L ER-CON10HT-1:ER-CON10HT-1 J5
 U 1 1 60D5C762
 P 7800 3500
-F 0 "J6" H 8300 3765 50  0000 C CNN
+F 0 "J5" H 8300 3765 50  0000 C CNN
 F 1 "ER-CON10HT-1" H 8300 3674 50  0000 C CNN
 F 2 "ER-CONNECTOR:ER-CON10HT1" H 8650 3600 50  0001 L CNN
@@
 	1500 3600 1500 3800
 $Comp
-L power:+3V3 #PWR034
+L power:+3V3 #PWR043
 U 1 1 60E38299
 P 1050 3250
-F 0 "#PWR034" H 1050 3100 50  0001 C CNN
+F 0 "#PWR043" H 1050 3100 50  0001 C CNN
 F 1 "+3V3" H 1065 3423 50  0000 C CNN
 F 2 "" H 1050 3250 50  0001 C CNN
@@
 $EndComp
 $Comp
-L power:+5V #PWR032
+L power:+5V #PWR041
 U 1 1 60E38786
 P 800 3250
-F 0 "#PWR032" H 800 3100 50  0001 C CNN
+F 0 "#PWR041" H 800 3100 50  0001 C CNN
 F 1 "+5V" H 815 3423 50  0000 C CNN
 F 2 "" H 800 3250 50  0001 C CNN
@@
 F 2 "TPS61165DRVR:TPS61165DRVR" H 2600 2150 50  0001 L BNN
 F 3 "http://www.ti.com/general/docs/suppproductinfo.tsp?distId=26&gotoUrl=http%3A%2F%2Fwww.ti.com%2Flit%2Fgpn%2Ftps61165" H 2900 1700 50  0001 L BNN
+F 4 "2156-TPS61165DRVR-ND" H 2900 1700 50  0001 C CNN "Digikey#"
+F 5 "Texas Instruments" H 2900 1700 50  0001 C CNN "MANUFACTURER"
+F 6 "TPS61165DRVR" H 2900 1700 50  0001 C CNN "Manf#"
+F 7 "595-TPS61165DRVR" H 2900 1700 50  0001 C CNN "Mouser#"
 	1    2900 1700
 	1    0    0    -1
 $EndComp
 $Comp
-L power:GND1 #PWR035
+L power:GND1 #PWR045
 U 1 1 60E59FED
 P 2950 2500
-F 0 "#PWR035" H 2950 2250 50  0001 C CNN
+F 0 "#PWR045" H 2950 2250 50  0001 C CNN
 F 1 "GND1" H 2955 2327 50  0000 C CNN
 F 2 "" H 2950 2500 50  0001 C CNN
@@
 	3450 1700 3750 1700
 $Comp
-L Device:C C38
+L Device:C C42
 U 1 1 60E6C733
 P 1650 1900
-F 0 "C38" H 1300 1950 50  0000 L CNN
+F 0 "C42" H 1300 1950 50  0000 L CNN
 F 1 "4.7uF" H 1300 1850 50  0000 L CNN
 F 2 "Capacitor_SMD:C_0603_1608Metric" H 1688 1750 50  0001 C CNN
@@
 	1650 1400 2250 1400
 $Comp
-L Device:C C39
+L Device:C C43
 U 1 1 60E74CAB
 P 2400 2250
-F 0 "C39" H 2515 2296 50  0000 L CNN
+F 0 "C43" H 2515 2296 50  0000 L CNN
 F 1 "220nF" H 2515 2205 50  0000 L CNN
 F 2 "Capacitor_SMD:C_0603_1608Metric" H 2438 2100 50  0001 C CNN
@@
 Connection ~ 1650 2400
 $Comp
-L power:GNDD #PWR033
+L power:GNDD #PWR042
 U 1 1 60E91830
 P 900 2400
-F 0 "#PWR033" H 900 2150 50  0001 C CNN
+F 0 "#PWR042" H 900 2150 50  0001 C CNN
 F 1 "GNDD" V 904 2290 50  0000 R CNN
 F 2 "" H 900 2400 50  0001 C CNN
@@
 	2250 1400 2400 1400
 $Comp
-L Device:R R3
+L Device:R R8
 U 1 1 60E9B7AB
 P 3750 1900
-F 0 "R3" H 3820 1946 50  0000 L CNN
+F 0 "R8" H 3820 1946 50  0000 L CNN
 F 1 "5.1 (1%)" H 3820 1855 50  0000 L CNN
 F 2 "" V 3680 1900 50  0001 C CNN
@@
 Connection ~ 3450 2400
 $Comp
-L Device:C C42
+L Device:C C46
 U 1 1 60EA46A4
 P 4300 1900
-F 0 "C42" H 4415 1946 50  0000 L CNN
+F 0 "C46" H 4415 1946 50  0000 L CNN
 F 1 "1uF" H 4415 1855 50  0000 L CNN
 F 2 "Capacitor_SMD:C_0603_1608Metric" H 4338 1750 50  0001 C CNN
@@
 F 2 "Diode_SMD:D_SOD-323" H 4000 1400 50  0001 C CNN
 F 3 "https://www.diodes.com/assets/Datasheets/ZHCS400.pdf" H 4000 1400 50  0001 C CNN
+F 4 "ZHCS400CT-ND" H 4000 1400 50  0001 C CNN "Digikey#"
+F 5 "Diodes Incorporated" H 4000 1400 50  0001 C CNN "MANUFACTURER"
+F 6 "ZHCS400TA" H 4000 1400 50  0001 C CNN "Manf#"
+F 7 "522-ZHCS400TA" H 4000 1400 50  0001 C CNN "Mouser#"
 	1    4000 1400
 	-1   0    0    1
@@
 C42 and C44 must be ceramic\ncapacitor and low ESR
 $Comp
-L Device:CP C41
+L Device:CP C45
 U 1 1 60D62E33
 P 3850 3550
-F 0 "C41" H 3968 3596 50  0000 L CNN
+F 0 "C45" H 3968 3596 50  0000 L CNN
 F 1 "4.7uF" H 3968 3505 50  0000 L CNN
 F 2 "595D475X9016A2T:595D475X9016A2T" H 3888 3400 50  0001 C CNN
@@
 Connection ~ 3700 3400
 $Comp
-L Device:CP C44
+L Device:CP C48
 U 1 1 60D6FDC6
 P 9800 3050
-F 0 "C44" H 9918 3096 50  0000 L CNN
+F 0 "C48" H 9918 3096 50  0000 L CNN
 F 1 "4.7uF" H 9918 3005 50  0000 L CNN
 F 2 "595D475X9016A2T:595D475X9016A2T" H 9838 2900 50  0001 C CNN
@@
 	1650 2400 2400 2400
 $Comp
-L power:GND1 #PWR0101
+L power:GND1 #PWR044
 U 1 1 610260A2
 P 1750 950
-F 0 "#PWR0101" H 1750 700 50  0001 C CNN
+F 0 "#PWR044" H 1750 700 50  0001 C CNN
 F 1 "GND1" H 1755 777 50  0000 C CNN
 F 2 "" H 1750 950 50  0001 C CNN
@@
 $EndComp
 $Comp
-L power:PWR_FLAG #FLG0103
+L power:PWR_FLAG #FLG012
 U 1 1 61027249
 P 1750 850
-F 0 "#FLG0103" H 1750 925 50  0001 C CNN
+F 0 "#FLG012" H 1750 925 50  0001 C CNN
 F 1 "PWR_FLAG" H 1750 1023 50  0000 C CNN
 F 2 "" H 1750 850 50  0001 C CNN

Commit message: I filled more component to Kicost script
Parts:
- L4, L5: Digikey# (none) -> 490-7811-1-ND; MANUFACTURER (none) -> Murata Electronics; Manf# (none) -> BLM18AG601SH1D; Mouser# (none) -> 81-BLM18AG601SH1D
- L6: Digikey# (none) -> 490-16513-1-ND; MANUFACTURER (none) -> Murata Electronics; Manf# (none) -> #A915AY-100M=P3; Mouser# (none) -> 81-#A915AY-100M=P3
Changed lines of the file:
@@
 Sheet 4 8
 Title "LCD"
-Date "2021-06-19"
+Date "2021-08-24"
 Rev "Rev. 1"
 Comp "HardGFX"
@@
 F 1 "BLM18AG601SH1D" V 1260 1400 50  0000 C CNN
 F 2 "Inductor_SMD:L_0603_1608Metric" H 1350 1400 50  0001 C CNN
-F 3 "https://ar.mouser.com/datasheet/2/281/QNFA9101-1915702.pdf" H 1350 1400 50  0001 C CNN
+F 3 "https://www.murata.com/en-us/products/productdata/8796737273886/QNFA9101.pdf" H 1350 1400 50  0001 C CNN
+F 4 "490-7811-1-ND" H 1350 1400 50  0001 C CNN "Digikey#"
+F 5 "Murata Electronics" H 1350 1400 50  0001 C CNN "MANUFACTURER"
+F 6 "BLM18AG601SH1D" H 1350 1400 50  0001 C CNN "Manf#"
+F 7 "81-BLM18AG601SH1D" H 1350 1400 50  0001 C CNN "Mouser#"
 	1    1350 1400
 	0    1    1    0
@@
 F 1 "BLM18AG601SH1D" V 1600 2400 50  0000 C CNN
 F 2 "Inductor_SMD:L_0603_1608Metric" H 1350 2400 50  0001 C CNN
-F 3 "https://ar.mouser.com/datasheet/2/281/QNFA9101-1915702.pdf" H 1350 2400 50  0001 C CNN
+F 3 "https://www.murata.com/en-us/products/productdata/8796737273886/QNFA9101.pdf" H 1350 2400 50  0001 C CNN
+F 4 "490-7811-1-ND" H 1350 2400 50  0001 C CNN "Digikey#"
+F 5 "Murata Electronics" H 1350 2400 50  0001 C CNN "MANUFACTURER"
+F 6 "BLM18AG601SH1D" H 1350 2400 50  0001 C CNN "Manf#"
+F 7 "81-BLM18AG601SH1D" H 1350 2400 50  0001 C CNN "Mouser#"
 	1    1350 2400
 	0    1    1    0
@@
 F 2 "A915AY-100M_P3:IND_#A915AY-100M=P3" H 2900 950 50  0001 C CNN
 F 3 "https://www.murata.com/en-global/api/pdfdownloadapi?cate=cgInductors&partno=%23A915AY-100M%3DP3" H 2900 950 50  0001 C CNN
+F 4 "490-16513-1-ND" H 2900 950 50  0001 C CNN "Digikey#"
+F 5 "Murata Electronics" H 2900 950 50  0001 C CNN "MANUFACTURER"
+F 6 "#A915AY-100M=P3" H 2900 950 50  0001 C CNN "Manf#"
+F 7 "81-#A915AY-100M=P3" H 2900 950 50  0001 C CNN "Mouser#"
 	1    2900 950
 	0    1    1    0

Commit message: Almost I end to fill Kicost field on schematics.
Parts:
- C42: Digikey# (none) -> 490-14373-1-ND; MANUFACTURER (none) -> Murata Electronics; Manf# (none) -> GRM188R61A475KAAJJ; Mouser# (none) -> 81-GRM188R61A475KAJJ
- C44, C47: Digikey# (none) -> 311-1088-1-ND; MANUFACTURER (none) -> YAGEO; Manf# (none) -> CC0603KRX7R7BB104; Mouser# (none) -> 603-CC603KRX7R7BB104
- C45, C48: Digikey# (none) -> 718-595D475X9016A2TCT-ND; MANUFACTURER (none) -> Vishay / Sprague; Manf# (none) -> 595D475X9016A2T; Mouser# (none) -> 74-595D475X9016A2T
- C46: Digikey# (none) -> 490-GRM188R61E105KAADJTR-ND; MANUFACTURER (none) -> Murata Electronics; Manf# (none) -> GRM188R61E105KAADJ; Mouser# (none) -> 81-GRM188R61E105KADJ
- J4, J5, JP10, JP9: Digikey# (none) -> -; MANUFACTURER (none) -> -; Manf# (none) -> -; Mouser# (none) -> -
- R9: Digikey# (none) -> 311-4.70KHRCT-ND; MANUFACTURER (none) -> YAGEO; Manf# (none) -> RC0603FR-074K7L; Mouser# (none) -> 603-RC0603FR-074K7L
Changed lines of the file:
@@
 Sheet 4 8
 Title "LCD"
-Date "2021-08-24"
+Date "2021-08-25"
 Rev "Rev. 1"
 Comp "HardGFX"
@@
 F 1 "100nF" H 3200 3500 50  0000 L CNN
 F 2 "Capacitor_SMD:C_0603_1608Metric" H 3588 3400 50  0001 C CNN
-F 3 "https://ar.mouser.com/datasheet/2/447/UPY_GPHC_X7R_6_3V_to_50V_20-1995650.pdf" H 3550 3550 50  0001 C CNN
+F 3 "https://www.yageo.com/upload/media/product/productsearch/datasheet/mlcc/UPY-GPHC_X7R_6.3V-to-50V_18.pdf" H 3550 3550 50  0001 C CNN
+F 4 "311-1088-1-ND" H 3550 3550 50  0001 C CNN "Digikey#"
+F 5 "YAGEO" H 3550 3550 50  0001 C CNN "MANUFACTURER"
+F 6 "CC0603KRX7R7BB104" H 3550 3550 50  0001 C CNN "Manf#"
+F 7 "603-CC603KRX7R7BB104" H 3550 3550 50  0001 C CNN "Mouser#"
 	1    3550 3550
 	1    0    0    -1
@@
 F 1 "4.7K" H 5070 6555 50  0000 L CNN
 F 2 "" V 4930 6600 50  0001 C CNN
-F 3 "~" H 5000 6600 50  0001 C CNN
+F 3 "https://www.yageo.com/upload/media/product/productsearch/datasheet/rchip/PYu-RC_Group_51_RoHS_L_11.pdf" H 5000 6600 50  0001 C CNN
+F 4 "311-4.70KHRCT-ND" H 5000 6600 50  0001 C CNN "Digikey#"
+F 5 "YAGEO" H 5000 6600 50  0001 C CNN "MANUFACTURER"
+F 6 "RC0603FR-074K7L" H 5000 6600 50  0001 C CNN "Manf#"
+F 7 "603-RC0603FR-074K7L" H 5000 6600 50  0001 C CNN "Mouser#"
 	1    5000 6600
 	1    0    0    -1
@@
 F 2 "ER-CONNECTOR:ER-CON40HT-1" H 5500 3100 50  0001 L BNN
 F 3 "https://www.buydisplay.com/download/connector/ER-CON40HT-1.pdf" H 5500 3100 50  0001 L BNN
+F 4 "-" H 5500 3100 50  0001 C CNN "Digikey#"
+F 5 "-" H 5500 3100 50  0001 C CNN "MANUFACTURER"
+F 6 "-" H 5500 3100 50  0001 C CNN "Manf#"
+F 7 "-" H 5500 3100 50  0001 C CNN "Mouser#"
 	1    5500 3100
 	1    0    0    -1
@@
 F 1 "100nF" H 9150 3000 50  0000 L CNN
 F 2 "Capacitor_SMD:C_0603_1608Metric" H 9538 2900 50  0001 C CNN
-F 3 "https://ar.mouser.com/datasheet/2/447/UPY_GPHC_X7R_6_3V_to_50V_20-1995650.pdf" H 9500 3050 50  0001 C CNN
+F 3 "https://www.yageo.com/upload/media/product/productsearch/datasheet/mlcc/UPY-GPHC_X7R_6.3V-to-50V_18.pdf" H 9500 3050 50  0001 C CNN
+F 4 "311-1088-1-ND" H 9500 3050 50  0001 C CNN "Digikey#"
+F 5 "YAGEO" H 9500 3050 50  0001 C CNN "MANUFACTURER"
+F 6 "CC0603KRX7R7BB104" H 9500 3050 50  0001 C CNN "Manf#"
+F 7 "603-CC603KRX7R7BB104" H 9500 3050 50  0001 C CNN "Mouser#"
 	1    9500 3050
 	1    0    0    -1
@@
 F 2 "ER-CONNECTOR:ER-CON10HT1" H 8650 3600 50  0001 L CNN
 F 3 "https://www.buydisplay.com/download/connector/ER-CON10HT-1.pdf" H 8650 3500 50  0001 L CNN
+F 4 "-" H 7800 3500 50  0001 C CNN "Digikey#"
+F 5 "-" H 7800 3500 50  0001 C CNN "MANUFACTURER"
+F 6 "-" H 7800 3500 50  0001 C CNN "Manf#"
+F 7 "-" H 7800 3500 50  0001 C CNN "Mouser#"
 	1    7800 3500
 	1    0    0    -1
@@
 F 1 "3.3V" H 1350 3250 50  0000 C CNN
 F 2 "Jumper:SolderJumper-2_P1.3mm_Open_Pad1.0x1.5mm" H 1350 3400 50  0001 C CNN
-F 3 "~" H 1350 3400 50  0001 C CNN
+F 3 "-" H 1350 3400 50  0001 C CNN
+F 4 "-" H 1350 3400 50  0001 C CNN "Digikey#"
+F 5 "-" H 1350 3400 50  0001 C CNN "MANUFACTURER"
+F 6 "-" H 1350 3400 50  0001 C CNN "Manf#"
+F 7 "-" H 1350 3400 50  0001 C CNN "Mouser#"
 	1    1350 3400
 	1    0    0    -1
@@
 F 1 "5V (Default)" H 1350 3650 50  0000 C CNN
 F 2 "Jumper:SolderJumper-2_P1.3mm_Open_Pad1.0x1.5mm" H 1350 3800 50  0001 C CNN
-F 3 "~" H 1350 3800 50  0001 C CNN
+F 3 "-" H 1350 3800 50  0001 C CNN
+F 4 "-" H 1350 3800 50  0001 C CNN "Digikey#"
+F 5 "-" H 1350 3800 50  0001 C CNN "MANUFACTURER"
+F 6 "-" H 1350 3800 50  0001 C CNN "Manf#"
+F 7 "-" H 1350 3800 50  0001 C CNN "Mouser#"
 	1    1350 3800
 	1    0    0    -1
@@
 F 2 "Capacitor_SMD:C_0603_1608Metric" H 1688 1750 50  0001 C CNN
 F 3 "https://search.murata.co.jp/Ceramy/image/img/A01X/G101/ENG/GRM188R61A475KAAJ-01.pdf" H 1650 1900 50  0001 C CNN
+F 4 "490-14373-1-ND" H 1650 1900 50  0001 C CNN "Digikey#"
+F 5 "Murata Electronics" H 1650 1900 50  0001 C CNN "MANUFACTURER"
+F 6 "GRM188R61A475KAAJJ" H 1650 1900 50  0001 C CNN "Manf#"
+F 7 "81-GRM188R61A475KAJJ" H 1650 1900 50  0001 C CNN "Mouser#"
 	1    1650 1900
 	1    0    0    -1
@@
 F 2 "Capacitor_SMD:C_0603_1608Metric" H 4338 1750 50  0001 C CNN
 F 3 "https://ar.mouser.com/datasheet/2/281/1/GRM188R61E105KAAD_01A-1985793.pdf" H 4300 1900 50  0001 C CNN
+F 4 "490-GRM188R61E105KAADJTR-ND" H 4300 1900 50  0001 C CNN "Digikey#"
+F 5 "Murata Electronics" H 4300 1900 50  0001 C CNN "MANUFACTURER"
+F 6 "GRM188R61E105KAADJ" H 4300 1900 50  0001 C CNN "Manf#"
+F 7 "81-GRM188R61E105KADJ" H 4300 1900 50  0001 C CNN "Mouser#"
 	1    4300 1900
 	1    0    0    -1
@@
 F 1 "4.7uF" H 3968 3505 50  0000 L CNN
 F 2 "595D475X9016A2T:595D475X9016A2T" H 3888 3400 50  0001 C CNN
-F 3 "https://ar.mouser.com/datasheet/2/427/595d-1763504.pdf" H 3850 3550 50  0001 C CNN
+F 3 "https://www.vishay.com/docs/40007/595d.pdf" H 3850 3550 50  0001 C CNN
+F 4 "718-595D475X9016A2TCT-ND" H 3850 3550 50  0001 C CNN "Digikey#"
+F 5 "Vishay / Sprague" H 3850 3550 50  0001 C CNN "MANUFACTURER"
+F 6 "595D475X9016A2T" H 3850 3550 50  0001 C CNN "Manf#"
+F 7 "74-595D475X9016A2T" H 3850 3550 50  0001 C CNN "Mouser#"
 	1    3850 3550
 	1    0    0    -1
@@
 F 1 "4.7uF" H 9918 3005 50  0000 L CNN
 F 2 "595D475X9016A2T:595D475X9016A2T" H 9838 2900 50  0001 C CNN
-F 3 "https://ar.mouser.com/datasheet/2/427/595d-1763504.pdf" H 9800 3050 50  0001 C CNN
+F 3 "https://www.vishay.com/docs/40007/595d.pdf" H 9800 3050 50  0001 C CNN
+F 4 "718-595D475X9016A2TCT-ND" H 9800 3050 50  0001 C CNN "Digikey#"
+F 5 "Vishay / Sprague" H 9800 3050 50  0001 C CNN "MANUFACTURER"
+F 6 "595D475X9016A2T" H 9800 3050 50  0001 C CNN "Manf#"
+F 7 "74-595D475X9016A2T" H 9800 3050 50  0001 C CNN "Mouser#"
 	1    9800 3050
 	1    0    0    -1
