File: HardGFX_STM32H745/HardGFX_LCD.sch (KiCad schematic (older format))
At the start: 18 parts, among them J4 ER-CON40HT-1, J5 ER-CON10HT-1, U5 TPS61165DRVR

Commit message: Modified symbols field to use Kicost
Parts:
- C42: Manf# GRM188R61A475KAAJJ -> (none); manf# (none) -> GRM188R61A475KAAJJ
- C44, C47: Manf# CC0603KRX7R7BB104 -> (none); manf# (none) -> CC0603KRX7R7BB104
- C45, C48: Manf# 595D475X9016A2T -> (none); manf# (none) -> 595D475X9016A2T
- C46: Manf# GRM188R61E105KAADJ -> (none); manf# (none) -> GRM188R61E105KAADJ
- D2: Manf# ZHCS400TA -> (none); manf# (none) -> ZHCS400TA
- J4, J5: Manf# - -> (none)
- JP10, JP9: Manf# - -> (none); manf# (none) -> -
- L4, L5: Manf# BLM18AG601SH1D -> (none); manf# (none) -> BLM18AG601SH1D
- L6: Manf# #A915AY-100M=P3 -> (none); manf# (none) -> #A915AY-100M=P3
- R9: Manf# RC0603FR-074K7L -> (none); manf# (none) -> RC0603FR-074K7L
- U5: Manf# TPS61165DRVR -> (none); manf# (none) -> TPS61165DRVR
Changed lines of the file:
@@
 F 4 "311-1088-1-ND" H 3550 3550 50  0001 C CNN "Digikey#"
 F 5 "YAGEO" H 3550 3550 50  0001 C CNN "MANUFACTURER"
-F 6 "CC0603KRX7R7BB104" H 3550 3550 50  0001 C CNN "Manf#"
+F 6 "" H 3550 3550 50  0001 C CNN "Manf#"
 F 7 "603-CC603KRX7R7BB104" H 3550 3550 50  0001 C CNN "Mouser#"
+F 8 "CC0603KRX7R7BB104" H 3550 3550 50  0001 C CNN "manf#"
 	1    3550 3550
 	1    0    0    -1
@@
 F 4 "311-4.70KHRCT-ND" H 5000 6600 50  0001 C CNN "Digikey#"
 F 5 "YAGEO" H 5000 6600 50  0001 C CNN "MANUFACTURER"
-F 6 "RC0603FR-074K7L" H 5000 6600 50  0001 C CNN "Manf#"
+F 6 "" H 5000 6600 50  0001 C CNN "Manf#"
 F 7 "603-RC0603FR-074K7L" H 5000 6600 50  0001 C CNN "Mouser#"
+F 8 "RC0603FR-074K7L" H 5000 6600 50  0001 C CNN "manf#"
 	1    5000 6600
 	1    0    0    -1
@@
 F 4 "-" H 5500 3100 50  0001 C CNN "Digikey#"
 F 5 "-" H 5500 3100 50  0001 C CNN "MANUFACTURER"
-F 6 "-" H 5500 3100 50  0001 C CNN "Manf#"
+F 6 "" H 5500 3100 50  0001 C CNN "Manf#"
 F 7 "-" H 5500 3100 50  0001 C CNN "Mouser#"
 	1    5500 3100
@@
 F 4 "311-1088-1-ND" H 9500 3050 50  0001 C CNN "Digikey#"
 F 5 "YAGEO" H 9500 3050 50  0001 C CNN "MANUFACTURER"
-F 6 "CC0603KRX7R7BB104" H 9500 3050 50  0001 C CNN "Manf#"
+F 6 "" H 9500 3050 50  0001 C CNN "Manf#"
 F 7 "603-CC603KRX7R7BB104" H 9500 3050 50  0001 C CNN "Mouser#"
+F 8 "CC0603KRX7R7BB104" H 9500 3050 50  0001 C CNN "manf#"
 	1    9500 3050
 	1    0    0    -1
@@
 F 4 "-" H 7800 3500 50  0001 C CNN "Digikey#"
 F 5 "-" H 7800 3500 50  0001 C CNN "MANUFACTURER"
-F 6 "-" H 7800 3500 50  0001 C CNN "Manf#"
+F 6 "" H 7800 3500 50  0001 C CNN "Manf#"
 F 7 "-" H 7800 3500 50  0001 C CNN "Mouser#"
 	1    7800 3500
@@
 F 4 "-" H 1350 3400 50  0001 C CNN "Digikey#"
 F 5 "-" H 1350 3400 50  0001 C CNN "MANUFACTURER"
-F 6 "-" H 1350 3400 50  0001 C CNN "Manf#"
+F 6 "" H 1350 3400 50  0001 C CNN "Manf#"
 F 7 "-" H 1350 3400 50  0001 C CNN "Mouser#"
+F 8 "-" H 1350 3400 50  0001 C CNN "manf#"
 	1    1350 3400
 	1    0    0    -1
@@
 F 4 "-" H 1350 3800 50  0001 C CNN "Digikey#"
 F 5 "-" H 1350 3800 50  0001 C CNN "MANUFACTURER"
-F 6 "-" H 1350 3800 50  0001 C CNN "Manf#"
+F 6 "" H 1350 3800 50  0001 C CNN "Manf#"
 F 7 "-" H 1350 3800 50  0001 C CNN "Mouser#"
+F 8 "-" H 1350 3800 50  0001 C CNN "manf#"
 	1    1350 3800
 	1    0    0    -1
@@
 F 4 "2156-TPS61165DRVR-ND" H 2900 1700 50  0001 C CNN "Digikey#"
 F 5 "Texas Instruments" H 2900 1700 50  0001 C CNN "MANUFACTURER"
-F 6 "TPS61165DRVR" H 2900 1700 50  0001 C CNN "Manf#"
+F 6 "" H 2900 1700 50  0001 C CNN "Manf#"
 F 7 "595-TPS61165DRVR" H 2900 1700 50  0001 C CNN "Mouser#"
+F 8 "TPS61165DRVR" H 2900 1700 50  0001 C CNN "manf#"
 	1    2900 1700
 	1    0    0    -1
@@
 F 4 "490-14373-1-ND" H 1650 1900 50  0001 C CNN "Digikey#"
 F 5 "Murata Electronics" H 1650 1900 50  0001 C CNN "MANUFACTURER"
-F 6 "GRM188R61A475KAAJJ" H 1650 1900 50  0001 C CNN "Manf#"
-F 7 "81-GRM188R61A475KAJJ" H 1650 1900 50  0001 C CNN "Mouser#"
+F 6 "81-GRM188R61A475KAJJ" H 1650 1900 50  0001 C CNN "Mouser#"
+F 7 "GRM188R61A475KAAJJ" H 1650 1900 50  0001 C CNN "manf#"
 	1    1650 1900
 	1    0    0    -1
@@
 F 4 "490-7811-1-ND" H 1350 1400 50  0001 C CNN "Digikey#"
 F 5 "Murata Electronics" H 1350 1400 50  0001 C CNN "MANUFACTURER"
-F 6 "BLM18AG601SH1D" H 1350 1400 50  0001 C CNN "Manf#"
-F 7 "81-BLM18AG601SH1D" H 1350 1400 50  0001 C CNN "Mouser#"
+F 6 "81-BLM18AG601SH1D" H 1350 1400 50  0001 C CNN "Mouser#"
+F 7 "BLM18AG601SH1D" H 1350 1400 50  0001 C CNN "manf#"
 	1    1350 1400
 	0    1    1    0
@@
 F 4 "490-7811-1-ND" H 1350 2400 50  0001 C CNN "Digikey#"
 F 5 "Murata Electronics" H 1350 2400 50  0001 C CNN "MANUFACTURER"
-F 6 "BLM18AG601SH1D" H 1350 2400 50  0001 C CNN "Manf#"
-F 7 "81-BLM18AG601SH1D" H 1350 2400 50  0001 C CNN "Mouser#"
+F 6 "81-BLM18AG601SH1D" H 1350 2400 50  0001 C CNN "Mouser#"
+F 7 "BLM18AG601SH1D" H 1350 2400 50  0001 C CNN "manf#"
 	1    1350 2400
 	0    1    1    0
@@
 F 4 "490-16513-1-ND" H 2900 950 50  0001 C CNN "Digikey#"
 F 5 "Murata Electronics" H 2900 950 50  0001 C CNN "MANUFACTURER"
-F 6 "#A915AY-100M=P3" H 2900 950 50  0001 C CNN "Manf#"
+F 6 "" H 2900 950 50  0001 C CNN "Manf#"
 F 7 "81-#A915AY-100M=P3" H 2900 950 50  0001 C CNN "Mouser#"
+F 8 "#A915AY-100M=P3" H 2900 950 50  0001 C CNN "manf#"
 	1    2900 950
 	0    1    1    0
@@
 F 4 "490-GRM188R61E105KAADJTR-ND" H 4300 1900 50  0001 C CNN "Digikey#"
 F 5 "Murata Electronics" H 4300 1900 50  0001 C CNN "MANUFACTURER"
-F 6 "GRM188R61E105KAADJ" H 4300 1900 50  0001 C CNN "Manf#"
+F 6 "" H 4300 1900 50  0001 C CNN "Manf#"
 F 7 "81-GRM188R61E105KADJ" H 4300 1900 50  0001 C CNN "Mouser#"
+F 8 "GRM188R61E105KAADJ" H 4300 1900 50  0001 C CNN "manf#"
 	1    4300 1900
 	1    0    0    -1
@@
 F 4 "ZHCS400CT-ND" H 4000 1400 50  0001 C CNN "Digikey#"
 F 5 "Diodes Incorporated" H 4000 1400 50  0001 C CNN "MANUFACTURER"
-F 6 "ZHCS400TA" H 4000 1400 50  0001 C CNN "Manf#"
+F 6 "" H 4000 1400 50  0001 C CNN "Manf#"
 F 7 "522-ZHCS400TA" H 4000 1400 50  0001 C CNN "Mouser#"
+F 8 "ZHCS400TA" H 4000 1400 50  0001 C CNN "manf#"
 	1    4000 1400
 	-1   0    0    1
@@
 F 4 "718-595D475X9016A2TCT-ND" H 3850 3550 50  0001 C CNN "Digikey#"
 F 5 "Vishay / Sprague" H 3850 3550 50  0001 C CNN "MANUFACTURER"
-F 6 "595D475X9016A2T" H 3850 3550 50  0001 C CNN "Manf#"
+F 6 "" H 3850 3550 50  0001 C CNN "Manf#"
 F 7 "74-595D475X9016A2T" H 3850 3550 50  0001 C CNN "Mouser#"
+F 8 "595D475X9016A2T" H 3850 3550 50  0001 C CNN "manf#"
 	1    3850 3550
 	1    0    0    -1
@@
 F 4 "718-595D475X9016A2TCT-ND" H 9800 3050 50  0001 C CNN "Digikey#"
 F 5 "Vishay / Sprague" H 9800 3050 50  0001 C CNN "MANUFACTURER"
-F 6 "595D475X9016A2T" H 9800 3050 50  0001 C CNN "Manf#"
+F 6 "" H 9800 3050 50  0001 C CNN "Manf#"
 F 7 "74-595D475X9016A2T" H 9800 3050 50  0001 C CNN "Mouser#"
+F 8 "595D475X9016A2T" H 9800 3050 50  0001 C CNN "manf#"
 	1    9800 3050
 	1    0    0    -1
