File: HardGFX_STM32H745/HardGFX_STM32H745.sch (KiCad schematic (older format))
At the start: 16 parts, among them SW1 SW_MEC_5E, U1 STM32H745BIT6, X1 25MHz, Y1 ECS-.327-6-34R-TR

Commit message: Modified symbols field to use Kicost
Parts:
- C1, C4: Manf# CC0603KRX7R7BB104 -> (none); manf# (none) -> CC0603KRX7R7BB104
- C2, C3: Manf# CC0603CRNPO9BN1R5 -> (none); manf# (none) -> CC0603CRNPO9BN1R5
- CR1: Manf# ESDA7P60-1U1M -> (none); manf# (none) -> ESDA7P60-1U1M
- R1, R2, R5: Manf# RC0603FR-0710KL -> (none); manf# (none) -> RC0603FR-0710KL
- R3, R4: Manf# RC0603FR-071K5L -> (none); manf# (none) -> RC0603FR-071K5L
- S1: Manf# CAS-D20TA -> (none); manf# (none) -> CAS-D20TA
- SW1: Manf# 430481025816 -> (none); manf# (none) -> 430481025816
- TP1: Manf# - -> (none); manf# (none) -> -
- U1: Manf# STM32H745BIT6 -> (none); manf# (none) -> STM32H745BIT6
- X1: Manf# ECS-2520MVQ-250-BS-TR -> (none); manf# (none) -> ECS-2520MVQ-250-BS-TR
- Y1: Manf# ABS07-LR-32.768KHZ-6-1-T -> (none); manf# (none) -> ABS07-LR-32.768KHZ-6-1-T
Changed lines of the file:
@@
 F 2 "STM32H745BIT3:STM32H745BIT3" H 3850 3540 60  0001 C CNN
 F 3 "https://www.st.com/resource/en/datasheet/stm32h745bi.pdf" H 2650 3300 60  0001 C CNN
-F 4 "STM32H745BIT6" H 2650 3300 50  0001 C CNN "Manf#"
-F 5 "STM32H745BIT6-ND" H 2650 3300 50  0001 C CNN "Digikey#"
-F 6 "STMicroelectronics" H 2650 3300 50  0001 C CNN "MANUFACTURER"
-F 7 "511-STM32H745BIT6" H 2650 3300 50  0001 C CNN "Mouser#"
+F 4 "STM32H745BIT6-ND" H 2650 3300 50  0001 C CNN "Digikey#"
+F 5 "STMicroelectronics" H 2650 3300 50  0001 C CNN "MANUFACTURER"
+F 6 "511-STM32H745BIT6" H 2650 3300 50  0001 C CNN "Mouser#"
+F 7 "STM32H745BIT6" H 2650 3300 50  0001 C CNN "manf#"
 	1    2650 3300
 	1    0    0    -1
@@
 F 2 "STM32H745BIT3:STM32H745BIT3" H 4150 8190 60  0001 C CNN
 F 3 "https://www.st.com/resource/en/datasheet/stm32h745bi.pdf" H 2950 7950 60  0001 C CNN
-F 4 "STM32H745BIT6" H 2950 7950 50  0001 C CNN "Manf#"
-F 5 "STM32H745BIT6-ND" H 2950 7950 50  0001 C CNN "Digikey#"
-F 6 "STMicroelectronics" H 2950 7950 50  0001 C CNN "MANUFACTURER"
-F 7 "511-STM32H745BIT6" H 2950 7950 50  0001 C CNN "Mouser#"
+F 4 "STM32H745BIT6-ND" H 2950 7950 50  0001 C CNN "Digikey#"
+F 5 "STMicroelectronics" H 2950 7950 50  0001 C CNN "MANUFACTURER"
+F 6 "511-STM32H745BIT6" H 2950 7950 50  0001 C CNN "Mouser#"
+F 7 "STM32H745BIT6" H 2950 7950 50  0001 C CNN "manf#"
 	3    2950 7950
 	1    0    0    -1
@@
 F 4 "311-1.50KHRCT-ND" H 5950 5950 50  0001 C CNN "Digikey#"
 F 5 "YAGEO" H 5950 5950 50  0001 C CNN "MANUFACTURER"
-F 6 "RC0603FR-071K5L" H 5950 5950 50  0001 C CNN "Manf#"
-F 7 "603-RC0603FR-071K5L" H 5950 5950 50  0001 C CNN "Mouser#"
+F 6 "603-RC0603FR-071K5L" H 5950 5950 50  0001 C CNN "Mouser#"
+F 7 "RC0603FR-071K5L" H 5950 5950 50  0001 C CNN "manf#"
 	1    5950 5950
 	1    0    0    -1
@@
 F 4 "311-1.50KHRCT-ND" H 6350 5950 50  0001 C CNN "Digikey#"
 F 5 "YAGEO" H 6350 5950 50  0001 C CNN "MANUFACTURER"
-F 6 "RC0603FR-071K5L" H 6350 5950 50  0001 C CNN "Manf#"
-F 7 "603-RC0603FR-071K5L" H 6350 5950 50  0001 C CNN "Mouser#"
+F 6 "603-RC0603FR-071K5L" H 6350 5950 50  0001 C CNN "Mouser#"
+F 7 "RC0603FR-071K5L" H 6350 5950 50  0001 C CNN "manf#"
 	1    6350 5950
 	1    0    0    -1
@@
 F 7 "2.5 mm" H 4350 10400 50  0001 L BNN "MAXIMUM_PACKAGE_HEIGHT"
 F 8 "CASD20JCT-ND" H 4350 10400 50  0001 C CNN "Digikey#"
-F 9 "CAS-D20TA" H 4350 10400 50  0001 C CNN "Manf#"
-F 10 "229-CAS-D20TA" H 4350 10400 50  0001 C CNN "Mouser#"
+F 9 "229-CAS-D20TA" H 4350 10400 50  0001 C CNN "Mouser#"
+F 10 "CAS-D20TA" H 4350 10400 50  0001 C CNN "manf#"
 	1    4350 10400
 	-1   0    0    1
@@
 F 4 "311-10.0KHRCT-ND" H 4950 9700 50  0001 C CNN "Digikey#"
 F 5 "YAGEO" H 4950 9700 50  0001 C CNN "MANUFACTURER"
-F 6 "RC0603FR-0710KL" H 4950 9700 50  0001 C CNN "Manf#"
-F 7 "603-RC0603FR-0710KL" H 4950 9700 50  0001 C CNN "Mouser#"
+F 6 "603-RC0603FR-0710KL" H 4950 9700 50  0001 C CNN "Mouser#"
+F 7 "RC0603FR-0710KL" H 4950 9700 50  0001 C CNN "manf#"
 	1    4950 9700
 	1    0    0    -1
@@
 F 4 "311-10.0KHRCT-ND" H 5350 9700 50  0001 C CNN "Digikey#"
 F 5 "YAGEO" H 5350 9700 50  0001 C CNN "MANUFACTURER"
-F 6 "RC0603FR-0710KL" H 5350 9700 50  0001 C CNN "Manf#"
-F 7 "603-RC0603FR-0710KL" H 5350 9700 50  0001 C CNN "Mouser#"
+F 6 "603-RC0603FR-0710KL" H 5350 9700 50  0001 C CNN "Mouser#"
+F 7 "RC0603FR-0710KL" H 5350 9700 50  0001 C CNN "manf#"
 	1    5350 9700
 	1    0    0    -1
@@
 F 4 "732-7022-1-ND" H 6900 9150 50  0001 C CNN "Digikey#"
 F 5 "Wurth Elektronik " H 6900 9150 50  0001 C CNN "MANUFACTURER"
-F 6 "430481025816" H 6900 9150 50  0001 C CNN "Manf#"
-F 7 "710-430481025816" H 6900 9150 50  0001 C CNN "Mouser#"
+F 6 "710-430481025816" H 6900 9150 50  0001 C CNN "Mouser#"
+F 7 "430481025816" H 6900 9150 50  0001 C CNN "manf#"
 	1    6900 9150
 	1    0    0    -1
@@
 F 4 "311-1088-1-ND" H 6000 9350 50  0001 C CNN "Digikey#"
 F 5 "YAGEO" H 6000 9350 50  0001 C CNN "MANUFACTURER"
-F 6 "CC0603KRX7R7BB104" H 6000 9350 50  0001 C CNN "Manf#"
-F 7 "603-CC603KRX7R7BB104" H 6000 9350 50  0001 C CNN "Mouser#"
+F 6 "603-CC603KRX7R7BB104" H 6000 9350 50  0001 C CNN "Mouser#"
+F 7 "CC0603KRX7R7BB104" H 6000 9350 50  0001 C CNN "manf#"
 	1    6000 9350
 	1    0    0    -1
@@
 F 4 "497-16253-1-ND" H 6700 9450 50  0001 C CNN "Digikey#"
 F 5 "STMicroelectronics" H 6700 9450 50  0001 C CNN "MANUFACTURER"
-F 6 "ESDA7P60-1U1M" H 6700 9450 50  0001 C CNN "Manf#"
-F 7 "511-ESDA7P60-1U1M" H 6700 9450 50  0001 C CNN "Mouser#"
+F 6 "511-ESDA7P60-1U1M" H 6700 9450 50  0001 C CNN "Mouser#"
+F 7 "ESDA7P60-1U1M" H 6700 9450 50  0001 C CNN "manf#"
 	1    6700 9450
 	1    0    0    -1
@@
 F 4 "535-12943-1-ND" H 7950 5300 50  0001 C CNN "Digikey#"
 F 5 "815-ABS07LR32.76-61T" H 7950 5300 50  0001 C CNN "Mouser#"
-F 6 "ABS07-LR-32.768KHZ-6-1-T" H 7950 5300 50  0001 C CNN "Manf#"
-F 7 "ABRACON" H 7950 5300 50  0001 C CNN "MANUFACTURER"
+F 6 "ABRACON" H 7950 5300 50  0001 C CNN "MANUFACTURER"
+F 7 "ABS07-LR-32.768KHZ-6-1-T" H 7950 5300 50  0001 C CNN "manf#"
 	1    7950 5300
 	1    0    0    -1
@@
 F 3 "https://ecsxtal.com/store/pdf/ECS-2520MVQ.pdf" H 14600 5450 50  0001 C CNN
 F 4 "50-ECS-2520MVQ-250-BS-CT-ND" H 14700 5450 50  0001 C CNN "Digikey#"
-F 5 "ECS-2520MVQ-250-BS-TR" H 14700 5450 50  0001 C CNN "Manf#"
-F 6 "520-2520MVQ-250-BSTR" H 14700 5450 50  0001 C CNN "Mouser#"
-F 7 "ECS" H 14700 5450 50  0001 C CNN "MANUFACTURER"
+F 5 "520-2520MVQ-250-BSTR" H 14700 5450 50  0001 C CNN "Mouser#"
+F 6 "ECS" H 14700 5450 50  0001 C CNN "MANUFACTURER"
+F 7 "ECS-2520MVQ-250-BS-TR" H 14700 5450 50  0001 C CNN "manf#"
 	1    14700 5450
 	0    -1   -1   0
@@
 F 4 "311-1050-1-ND" H 7500 5650 50  0001 C CNN "Digikey#"
 F 5 "YAGEO" H 7500 5650 50  0001 C CNN "MANUFACTURER"
-F 6 "CC0603CRNPO9BN1R5" H 7500 5650 50  0001 C CNN "Manf#"
-F 7 "603-CC603CRNPO9BN1R5" H 7500 5650 50  0001 C CNN "Mouser#"
+F 6 "603-CC603CRNPO9BN1R5" H 7500 5650 50  0001 C CNN "Mouser#"
+F 7 "CC0603CRNPO9BN1R5" H 7500 5650 50  0001 C CNN "manf#"
 	1    7500 5650
 	1    0    0    -1
@@
 F 4 "311-1050-1-ND" H 8400 5650 50  0001 C CNN "Digikey#"
 F 5 "YAGEO" H 8400 5650 50  0001 C CNN "MANUFACTURER"
-F 6 "CC0603CRNPO9BN1R5" H 8400 5650 50  0001 C CNN "Manf#"
-F 7 "603-CC603CRNPO9BN1R5" H 8400 5650 50  0001 C CNN "Mouser#"
+F 6 "603-CC603CRNPO9BN1R5" H 8400 5650 50  0001 C CNN "Mouser#"
+F 7 "CC0603CRNPO9BN1R5" H 8400 5650 50  0001 C CNN "manf#"
 	1    8400 5650
 	1    0    0    -1
@@
 F 4 "311-1088-1-ND" H 14200 6150 50  0001 C CNN "Digikey#"
 F 5 "YAGEO" H 14200 6150 50  0001 C CNN "MANUFACTURER"
-F 6 "CC0603KRX7R7BB104" H 14200 6150 50  0001 C CNN "Manf#"
-F 7 "603-CC603KRX7R7BB104" H 14200 6150 50  0001 C CNN "Mouser#"
+F 6 "603-CC603KRX7R7BB104" H 14200 6150 50  0001 C CNN "Mouser#"
+F 7 "CC0603KRX7R7BB104" H 14200 6150 50  0001 C CNN "manf#"
 	1    14200 6150
 	1    0    0    -1
@@
 F 4 "311-10.0KHRCT-ND" H 14450 5850 50  0001 C CNN "Digikey#"
 F 5 "YAGEO" H 14450 5850 50  0001 C CNN "MANUFACTURER"
-F 6 "RC0603FR-0710KL" H 14450 5850 50  0001 C CNN "Manf#"
-F 7 "603-RC0603FR-0710KL" H 14450 5850 50  0001 C CNN "Mouser#"
+F 6 "603-RC0603FR-0710KL" H 14450 5850 50  0001 C CNN "Mouser#"
+F 7 "RC0603FR-0710KL" H 14450 5850 50  0001 C CNN "manf#"
 	1    14450 5850
 	0    1    1    0
@@
 F 4 "-" H 13450 5100 50  0001 C CNN "Digikey#"
 F 5 "-" H 13450 5100 50  0001 C CNN "MANUFACTURER"
-F 6 "-" H 13450 5100 50  0001 C CNN "Manf#"
+F 6 "" H 13450 5100 50  0001 C CNN "Manf#"
 F 7 "-" H 13450 5100 50  0001 C CNN "Mouser#"
+F 8 "-" H 13450 5100 50  0001 C CNN "manf#"
 	1    13450 5100
 	0    1    1    0
@@
 F 2 "STM32H745BIT3:STM32H745BIT3" H 11300 3540 60  0001 C CNN
 F 3 "https://www.st.com/resource/en/datasheet/stm32h745bi.pdf" H 10100 3300 60  0001 C CNN
-F 4 "STM32H745BIT6" H 10100 3300 50  0001 C CNN "Manf#"
-F 5 "STM32H745BIT6-ND" H 10100 3300 50  0001 C CNN "Digikey#"
-F 6 "STMicroelectronics" H 10100 3300 50  0001 C CNN "MANUFACTURER"
-F 7 "511-STM32H745BIT6" H 10100 3300 50  0001 C CNN "Mouser#"
+F 4 "STM32H745BIT6-ND" H 10100 3300 50  0001 C CNN "Digikey#"
+F 5 "STMicroelectronics" H 10100 3300 50  0001 C CNN "MANUFACTURER"
+F 6 "511-STM32H745BIT6" H 10100 3300 50  0001 C CNN "Mouser#"
+F 7 "STM32H745BIT6" H 10100 3300 50  0001 C CNN "manf#"
 	2    10100 3300
 	1    0    0    -1
