File: HardGFX_STM32H745/HardGFX_USB_WiFi.sch (KiCad schematic (older format))
At the start: 24 parts, among them J6 UART, J7 JTAG, J8 Boot Option, J9 47590-0001, Q1 BSR14, SW2 SW_MEC_5E, U10 STMPS2151STR, U11 USBLC6-4SC6, U9 ESP32-WROOM-32E_(4MB)

Commit message: Modified symbols field to use Kicost
Parts:
- C63, C66: Manf# CC0603KRX7R7BB104 -> (none); manf# (none) -> CC0603KRX7R7BB104
- C64: Manf# CC0603KRX5R7BB105 -> (none); manf# (none) -> CC0603KRX5R7BB105
- C67: Manf# 595D475X9016A2T -> (none); manf# (none) -> 595D475X9016A2T
- D3: Manf# 156120RS75000 -> (none); manf# (none) -> 156120RS75000
- D4: Manf# 156120VS75000 -> (none); manf# (none) -> 156120VS75000
- J6, J7: Manf# 54101-G1004LF -> (none); manf# (none) -> 54101-G1004LF
- J8: Manf# 54101-S0802LF -> (none); manf# (none) -> 54101-S0802LF
- J9: Manf# 47590-0001 -> (none); manf# (none) -> 47590-0001
- Q1: Manf# BSR14 -> (none); manf# (none) -> BSR14
- R11, R13: Manf# RC0603FR-0710KL -> (none); manf# (none) -> RC0603FR-0710KL
- R12: Manf# PMR03EZPJ000 -> (none); manf# (none) -> PMR03EZPJ000
- R14, R16: Manf# RC0603FR-0747KL -> (none); manf# (none) -> RC0603FR-0747KL
- R15: Manf# RC0603FR-07620RL -> (none); manf# (none) -> RC0603FR-07620RL
- R17: Manf# RC0603FR-0722KL -> (none); manf# (none) -> RC0603FR-0722KL
- R18: Manf# RC0603FR-07330RL -> (none); manf# (none) -> RC0603FR-07330RL
- SW2: Manf# 430481025816 -> (none); manf# (none) -> 430481025816
- U10: Manf# STMPS2151STR -> (none); manf# (none) -> STMPS2151STR
- U11: Manf# USBLC6-4SC6 -> (none); manf# (none) -> USBLC6-4SC6
- U9: Manf# ESP32-WROOM-32E (4MB HIGH TEMP) -> (none); manf# (none) -> ESP32-WROOM-32E (4MB HIGH TEMP)
Changed lines of the file:
@@
 F 6 "B1" H 10250 2500 50  0001 L BNN "PARTREV"
 F 7 "2266-47590-0001-ND" H 10200 3350 50  0001 C CNN "Digikey#"
-F 8 "47590-0001" H 10200 3350 50  0001 C CNN "Manf#"
+F 8 "" H 10200 3350 50  0001 C CNN "Manf#"
 F 9 "538-47590-0001" H 10200 3350 50  0001 C CNN "Mouser#"
+F 10 "47590-0001" H 10200 3350 50  0001 C CNN "manf#"
 	1    10200 3350
 	1    0    0    -1
@@
 F 3 "https://www.st.com/resource/en/datasheet/usblc6-4.pdf" H 8200 5150 50  0001 C CNN
 F 4 "497-4492-1-ND" H 8000 4800 50  0001 C CNN "Digikey#"
-F 5 "USBLC6-4SC6" H 8000 4800 50  0001 C CNN "Manf#"
+F 5 "" H 8000 4800 50  0001 C CNN "Manf#"
 F 6 "511-USBLC6-4SC6" H 8000 4800 50  0001 C CNN "Mouser#"
 F 7 "STMicroelectronics" H 8000 4800 50  0001 C CNN "MANUFACTURER"
+F 8 "USBLC6-4SC6" H 8000 4800 50  0001 C CNN "manf#"
 	1    8000 4800
 	1    0    0    -1
@@
 F 4 "497-6934-1-ND" H 7250 2450 50  0001 C CNN "Digikey#"
 F 5 "511-STMPS2151STR" H 7250 2450 50  0001 C CNN "Mouser#"
-F 6 "STMPS2151STR" H 7250 2450 50  0001 C CNN "Manf#"
+F 6 "" H 7250 2450 50  0001 C CNN "Manf#"
 F 7 "STMicroelectronics" H 7250 2450 50  0001 C CNN "MANUFACTURER"
+F 8 "STMPS2151STR" H 7250 2450 50  0001 C CNN "manf#"
 	1    7250 2450
 	1    0    0    -1
@@
 F 4 "311-10.0KHRCT-ND" H 7300 2750 50  0001 C CNN "Digikey#"
 F 5 "YAGEO" H 7300 2750 50  0001 C CNN "MANUFACTURER"
-F 6 "RC0603FR-0710KL" H 7300 2750 50  0001 C CNN "Manf#"
+F 6 "" H 7300 2750 50  0001 C CNN "Manf#"
 F 7 "603-RC0603FR-0710KL" H 7300 2750 50  0001 C CNN "Mouser#"
+F 8 "RC0603FR-0710KL" H 7300 2750 50  0001 C CNN "manf#"
 	1    7300 2750
 	1    0    0    -1
@@
 F 4 "718-595D475X9016A2TCT-ND" H 8900 2600 50  0001 C CNN "Digikey#"
 F 5 "Vishay / Sprague" H 8900 2600 50  0001 C CNN "MANUFACTURER"
-F 6 "595D475X9016A2T" H 8900 2600 50  0001 C CNN "Manf#"
+F 6 "" H 8900 2600 50  0001 C CNN "Manf#"
 F 7 "74-595D475X9016A2T" H 8900 2600 50  0001 C CNN "Mouser#"
+F 8 "595D475X9016A2T" H 8900 2600 50  0001 C CNN "manf#"
 	1    8900 2600
 	1    0    0    -1
@@
 F 4 "311-47.0KHRCT-ND" H 8700 1050 50  0001 C CNN "Digikey#"
 F 5 "YAGEO" H 8700 1050 50  0001 C CNN "MANUFACTURER"
-F 6 "RC0603FR-0747KL" H 8700 1050 50  0001 C CNN "Manf#"
+F 6 "" H 8700 1050 50  0001 C CNN "Manf#"
 F 7 "603-RC0603FR-0747KL" H 8700 1050 50  0001 C CNN "Mouser#"
+F 8 "RC0603FR-0747KL" H 8700 1050 50  0001 C CNN "manf#"
 	1    8700 1050
 	1    0    0    -1
@@
 F 4 "311-620HRCT-ND" H 9000 1050 50  0001 C CNN "Digikey#"
 F 5 "YAGEO" H 9000 1050 50  0001 C CNN "MANUFACTURER"
-F 6 "RC0603FR-07620RL" H 9000 1050 50  0001 C CNN "Manf#"
+F 6 "" H 9000 1050 50  0001 C CNN "Manf#"
 F 7 "603-RC0603FR-07620RL" H 9000 1050 50  0001 C CNN "Mouser#"
+F 8 "RC0603FR-07620RL" H 9000 1050 50  0001 C CNN "manf#"
 	1    9000 1050
 	1    0    0    -1
@@
 F 4 "732-5030-1-ND" H 9000 1450 50  0001 C CNN "Digikey#"
 F 5 "Wurth Elektronik" H 9000 1450 50  0001 C CNN "MANUFACTURER"
-F 6 "156120RS75000" H 9000 1450 50  0001 C CNN "Manf#"
+F 6 "" H 9000 1450 50  0001 C CNN "Manf#"
 F 7 "710-156120RS75000" H 9000 1450 50  0001 C CNN "Mouser#"
+F 8 "156120RS75000" H 9000 1450 50  0001 C CNN "manf#"
 	1    9000 1450
 	0    -1   -1   0
@@
 F 4 "311-330HRCT-ND" H 10250 4500 50  0001 C CNN "Digikey#"
 F 5 "YAGEO" H 10250 4500 50  0001 C CNN "MANUFACTURER"
-F 6 "RC0603FR-07330RL" H 10250 4500 50  0001 C CNN "Manf#"
+F 6 "" H 10250 4500 50  0001 C CNN "Manf#"
 F 7 "603-RC0603FR-07330RL" H 10250 4500 50  0001 C CNN "Mouser#"
+F 8 "RC0603FR-07330RL" H 10250 4500 50  0001 C CNN "manf#"
 	1    10250 4500
 	1    0    0    -1
@@
 F 4 "732-5032-1-ND" H 10250 4900 50  0001 C CNN "Digikey#"
 F 5 "Wurth Elektronik" H 10250 4900 50  0001 C CNN "MANUFACTURER"
-F 6 "156120VS75000" H 10250 4900 50  0001 C CNN "Manf#"
+F 6 "" H 10250 4900 50  0001 C CNN "Manf#"
 F 7 "710-156120VS75000" H 10250 4900 50  0001 C CNN "Mouser#"
+F 8 "156120VS75000" H 10250 4900 50  0001 C CNN "manf#"
 	1    10250 4900
 	0    -1   -1   0
@@
 F 4 "311-22.0KHRCT-ND" H 10000 5650 50  0001 C CNN "Digikey#"
 F 5 "YAGEO" H 10000 5650 50  0001 C CNN "MANUFACTURER"
-F 6 "RC0603FR-0722KL" H 10000 5650 50  0001 C CNN "Manf#"
+F 6 "" H 10000 5650 50  0001 C CNN "Manf#"
 F 7 "603-RC0603FR-0722KL" H 10000 5650 50  0001 C CNN "Mouser#"
+F 8 "RC0603FR-0722KL" H 10000 5650 50  0001 C CNN "manf#"
 	1    10000 5650
 	0    1    1    0
@@
 F 4 "311-47.0KHRCT-ND" H 9600 5350 50  0001 C CNN "Digikey#"
 F 5 "YAGEO" H 9600 5350 50  0001 C CNN "MANUFACTURER"
-F 6 "RC0603FR-0747KL" H 9600 5350 50  0001 C CNN "Manf#"
+F 6 "" H 9600 5350 50  0001 C CNN "Manf#"
 F 7 "603-RC0603FR-0747KL" H 9600 5350 50  0001 C CNN "Mouser#"
+F 8 "RC0603FR-0747KL" H 9600 5350 50  0001 C CNN "manf#"
 	1    9600 5350
 	0    1    1    0
@@
 F 7 "1965-ESP32-WROOM-32E(4MBHIGHTEMP)TR-ND" H 3350 4000 50  0001 C CNN "Digikey#"
 F 8 "356-ESP32WRM320EH3PS" H 3350 4000 50  0001 C CNN "Mouser#"
-F 9 "ESP32-WROOM-32E (4MB HIGH TEMP)" H 3350 4000 50  0001 C CNN "Manf#"
+F 9 "" H 3350 4000 50  0001 C CNN "Manf#"
 F 10 "Espressif Systems" H 3350 4000 50  0001 L BNN "MANUFACTURER"
+F 11 "ESP32-WROOM-32E (4MB HIGH TEMP)" H 3350 4000 50  0001 C CNN "manf#"
 	1    3350 4000
 	1    0    0    -1
@@
 F 4 "311-10.0KHRCT-ND" H 1600 2900 50  0001 C CNN "Digikey#"
 F 5 "YAGEO" H 1600 2900 50  0001 C CNN "MANUFACTURER"
-F 6 "RC0603FR-0710KL" H 1600 2900 50  0001 C CNN "Manf#"
+F 6 "" H 1600 2900 50  0001 C CNN "Manf#"
 F 7 "603-RC0603FR-0710KL" H 1600 2900 50  0001 C CNN "Mouser#"
+F 8 "RC0603FR-0710KL" H 1600 2900 50  0001 C CNN "manf#"
 	1    1600 2900
 	0    1    1    0
@@
 F 4 "311-1444-1-ND" H 2000 3050 50  0001 C CNN "Digikey#"
 F 5 "YAGEO" H 2000 3050 50  0001 C CNN "MANUFACTURER"
-F 6 "CC0603KRX5R7BB105" H 2000 3050 50  0001 C CNN "Manf#"
+F 6 "" H 2000 3050 50  0001 C CNN "Manf#"
 F 7 "603-CC603KRX5R7BB105" H 2000 3050 50  0001 C CNN "Mouser#"
+F 8 "CC0603KRX5R7BB105" H 2000 3050 50  0001 C CNN "manf#"
 	1    2000 3050
 	1    0    0    -1
@@
 F 4 "311-1088-1-ND" H 1900 2150 50  0001 C CNN "Digikey#"
 F 5 "YAGEO" H 1900 2150 50  0001 C CNN "MANUFACTURER"
-F 6 "CC0603KRX7R7BB104" H 1900 2150 50  0001 C CNN "Manf#"
+F 6 "" H 1900 2150 50  0001 C CNN "Manf#"
 F 7 "603-CC603KRX7R7BB104" H 1900 2150 50  0001 C CNN "Mouser#"
+F 8 "CC0603KRX7R7BB104" H 1900 2150 50  0001 C CNN "manf#"
 	1    1900 2150
 	0    1    1    0
@@
 F 4 "PMR03EZPJ000-ND" H 2250 2400 50  0001 C CNN "Digikey#"
 F 5 "ROHM Semiconductor" H 2250 2400 50  0001 C CNN "MANUFACTURER"
-F 6 "PMR03EZPJ000" H 2250 2400 50  0001 C CNN "Manf#"
+F 6 "" H 2250 2400 50  0001 C CNN "Manf#"
 F 7 "755-PMR03EZPJ000" H 2250 2400 50  0001 C CNN "Mouser#"
+F 8 "PMR03EZPJ000" H 2250 2400 50  0001 C CNN "manf#"
 	1    2250 2400
 	1    0    0    -1
@@
 F 4 "311-1088-1-ND" H 5600 2950 50  0001 C CNN "Digikey#"
 F 5 "YAGEO" H 5600 2950 50  0001 C CNN "MANUFACTURER"
-F 6 "CC0603KRX7R7BB104" H 5600 2950 50  0001 C CNN "Manf#"
+F 6 "" H 5600 2950 50  0001 C CNN "Manf#"
 F 7 "603-CC603KRX7R7BB104" H 5600 2950 50  0001 C CNN "Mouser#"
+F 8 "CC0603KRX7R7BB104" H 5600 2950 50  0001 C CNN "manf#"
 	1    5600 2950
 	1    0    0    -1
@@
 F 4 "54101-S0802LF-ND" H 5350 3700 50  0001 C CNN "Digikey#"
 F 5 "Amphenol FCI" H 5350 3700 50  0001 C CNN "MANUFACTURER"
-F 6 "54101-S0802LF" H 5350 3700 50  0001 C CNN "Manf#"
+F 6 "" H 5350 3700 50  0001 C CNN "Manf#"
 F 7 "649-54101-S0802LF" H 5350 3700 50  0001 C CNN "Mouser#"
+F 8 "54101-S0802LF" H 5350 3700 50  0001 C CNN "manf#"
 	1    5350 3700
 	1    0    0    -1
@@
 F 4 "54101-G1004LF-ND" H 1050 3750 50  0001 C CNN "Digikey#"
 F 5 "Amphenol FCI" H 1050 3750 50  0001 C CNN "MANUFACTURER"
-F 6 "54101-G1004LF" H 1050 3750 50  0001 C CNN "Manf#"
+F 6 "" H 1050 3750 50  0001 C CNN "Manf#"
 F 7 "649-54101-G1004LF" H 1050 3750 50  0001 C CNN "Mouser#"
+F 8 "54101-G1004LF" H 1050 3750 50  0001 C CNN "manf#"
 	1    1050 3750
 	-1   0    0    1
@@
 F 4 "54101-G1004LF-ND" H 5250 4350 50  0001 C CNN "Digikey#"
 F 5 "Amphenol FCI" H 5250 4350 50  0001 C CNN "MANUFACTURER"
-F 6 "54101-G1004LF" H 5250 4350 50  0001 C CNN "Manf#"
+F 6 "" H 5250 4350 50  0001 C CNN "Manf#"
 F 7 "649-54101-G1004LF" H 5250 4350 50  0001 C CNN "Mouser#"
+F 8 "54101-G1004LF" H 5250 4350 50  0001 C CNN "manf#"
 	1    5250 4350
 	1    0    0    -1
@@
 F 4 "732-7022-1-ND" H 1900 1900 50  0001 C CNN "Digikey#"
 F 5 "Wurth Elektronik " H 1900 1900 50  0001 C CNN "MANUFACTURER"
-F 6 "430481025816" H 1900 1900 50  0001 C CNN "Manf#"
+F 6 "" H 1900 1900 50  0001 C CNN "Manf#"
 F 7 "710-430481025816" H 1900 1900 50  0001 C CNN "Mouser#"
+F 8 "430481025816" H 1900 1900 50  0001 C CNN "manf#"
 	1    1900 1900
 	1    0    0    -1
@@
 F 4 "BSR14CT-ND" H 10150 5350 50  0001 C CNN "Digikey#"
 F 5 "onsemi / Fairchild" H 10150 5350 50  0001 C CNN "MANUFACTURER"
-F 6 "BSR14 " H 10150 5350 50  0001 C CNN "Manf#"
+F 6 "" H 10150 5350 50  0001 C CNN "Manf#"
 F 7 "512-BSR14" H 10150 5350 50  0001 C CNN "Mouser#"
+F 8 "BSR14 " H 10150 5350 50  0001 C CNN "manf#"
 	1    10150 5350
 	1    0    0    -1
